Commit message: Changed sensor kit parameters to fit the nissan leaf sensor kit.

File: nissan_leaf_sensor_kit_description/urdf/sensor_kit.xacro (robot description, xacro)
@@ -6,4 +6,6 @@
     <xacro:include filename="$(find camera_description)/urdf/monocular_camera.xacro"/>
     <xacro:include filename="$(find imu_description)/urdf/imu.xacro"/>
+    <xacro:include filename="$(find ouster_description)/urdf/OS1-64.urdf.xacro"/>
+    <xacro:include filename="$(find ouster_description)/urdf/OS2-64.urdf.xacro"/>
     <xacro:arg name="gpu" default="false"/>
     <xacro:arg name="config_dir" default="$(find nissan_leaf_sensor_kit_description)/config"/>
@@ -20,36 +22,26 @@
     <xacro:property name="calibration" value="${load_yaml('$(arg config_dir)/sensor_kit_calibration.yaml')}"/>
     <!-- lidar -->
-    <xacro:VLS-128 parent="sensor_kit_base_link" name="velodyne_top" topic="/points_raw" hz="10" samples="220" gpu="$(arg gpu)">
+    <xacro:OS1-64 parent="sensor_kit_base_link" name="lidar_os1/sensor" topic_points="/points" hz="10" samples="220">
       <origin
-        xyz="${calibration['sensor_kit_base_link']['velodyne_top_base_link']['x']}
-             ${calibration['sensor_kit_base_link']['velodyne_top_base_link']['y']}
-             ${calibration['sensor_kit_base_link']['velodyne_top_base_link']['z']}"
-        rpy="${calibration['sensor_kit_base_link']['velodyne_top_base_link']['roll']}
-             ${calibration['sensor_kit_base_link']['velodyne_top_base_link']['pitch']}
-             ${calibration['sensor_kit_base_link']['velodyne_top_base_link']['yaw']}"
+        xyz="${calibration['sensor_kit_base_link']['lidar_os1/sensor']['x']}
+             ${calibration['sensor_kit_base_link']['lidar_os1/sensor']['y']}
+             ${calibration['sensor_kit_base_link']['lidar_os1/sensor']['z']}"
+        rpy="${calibration['sensor_kit_base_link']['lidar_os1/sensor']['roll']}
+             ${calibration['sensor_kit_base_link']['lidar_os1/sensor']['pitch']}
+             ${calibration['sensor_kit_base_link']['lidar_os1/sensor']['yaw']}"
       />
-    </xacro:VLS-128>
-    <xacro:VLP-16 parent="sensor_kit_base_link" name="velodyne_left" topic="/points_raw" hz="10" samples="220" gpu="$(arg gpu)">
+    </xacro:OS1-64>
+    <xacro:OS2-64 parent="sensor_kit_base_link" name="lidar_os2/sensor" topic_points="/points" hz="10" samples="220">
       <origin
-        xyz="${calibration['sensor_kit_base_link']['velodyne_left_base_link']['x']}
-             ${calibration['sensor_kit_base_link']['velodyne_left_base_link']['y']}
-             ${calibration['sensor_kit_base_link']['velodyne_left_base_link']['z']}"
-        rpy="${calibration['sensor_kit_base_link']['velodyne_left_base_link']['roll']}
-             ${calibration['sensor_kit_base_link']['velodyne_left_base_link']['pitch']}
-             ${calibration['sensor_kit_base_link']['velodyne_left_base_link']['yaw']}"
+        xyz="${calibration['sensor_kit_base_link']['lidar_os2/sensor']['x']}
+             ${calibration['sensor_kit_base_link']['lidar_os2/sensor']['y']}
+             ${calibration['sensor_kit_base_link']['lidar_os2/sensor']['z']}"
+        rpy="${calibration['sensor_kit_base_link']['lidar_os2/sensor']['roll']}
+             ${calibration['sensor_kit_base_link']['lidar_os2/sensor']['pitch']}
+             ${calibration['sensor_kit_base_link']['lidar_os2/sensor']['yaw']}"
       />
-    </xacro:VLP-16>
-    <xacro:VLP-16 parent="sensor_kit_base_link" name="velodyne_right" topic="/points_raw" hz="10" samples="220" gpu="$(arg gpu)">
-      <origin
-        xyz="${calibration['sensor_kit_base_link']['velodyne_right_base_link']['x']}
-             ${calibration['sensor_kit_base_link']['velodyne_right_base_link']['y']}
-             ${calibration['sensor_kit_base_link']['velodyne_right_base_link']['z']}"
-        rpy="${calibration['sensor_kit_base_link']['velodyne_right_base_link']['roll']}
-             ${calibration['sensor_kit_base_link']['velodyne_right_base_link']['pitch']}
-             ${calibration['sensor_kit_base_link']['velodyne_right_base_link']['yaw']}"
-      />
-    </xacro:VLP-16>
+    </xacro:OS2-64>
     <!-- camera -->
-    <xacro:monocular_camera_macro
+<!--     <xacro:monocular_camera_macro
       name="traffic_light_right_camera/camera"
       parent="sensor_kit_base_link"
@@ -80,15 +72,15 @@
       height="400"
       fov="1.3"
-    />
+    /> -->
     <xacro:monocular_camera_macro
-      name="camera0/camera"
+      name="camera_front/camera"
       parent="sensor_kit_base_link"
       namespace=""
-      x="${calibration['sensor_kit_base_link']['camera0/camera_link']['x']}"
-      y="${calibration['sensor_kit_base_link']['camera0/camera_link']['y']}"
-      z="${calibration['sensor_kit_base_link']['camera0/camera_link']['z']}"
-      roll="${calibration['sensor_kit_base_link']['camera0/camera_link']['roll']}"
-      pitch="${calibration['sensor_kit_base_link']['camera0/camera_link']['pitch']}"
-      yaw="${calibration['sensor_kit_base_link']['camera0/camera_link']['yaw']}"
+      x="${calibration['sensor_kit_base_link']['camera_front/camera_link']['x']}"
+      y="${calibration['sensor_kit_base_link']['camera_front/camera_link']['y']}"
+      z="${calibration['sensor_kit_base_link']['camera_front/camera_link']['z']}"
+      roll="${calibration['sensor_kit_base_link']['camera_front/camera_link']['roll']}"
+      pitch="${calibration['sensor_kit_base_link']['camera_front/camera_link']['pitch']}"
+      yaw="${calibration['sensor_kit_base_link']['camera_front/camera_link']['yaw']}"
       fps="30"
       width="800"
@@ -97,13 +89,13 @@
     />
     <xacro:monocular_camera_macro
-      name="camera1/camera"
+      name="camera_rear/camera"
       parent="sensor_kit_base_link"
       namespace=""
-      x="${calibration['sensor_kit_base_link']['camera1/camera_link']['x']}"
-      y="${calibration['sensor_kit_base_link']['camera1/camera_link']['y']}"
-      z="${calibration['sensor_kit_base_link']['camera1/camera_link']['z']}"
-      roll="${calibration['sensor_kit_base_link']['camera1/camera_link']['roll']}"
-      pitch="${calibration['sensor_kit_base_link']['camera1/camera_link']['pitch']}"
-      yaw="${calibration['sensor_kit_base_link']['camera1/camera_link']['yaw']}"
+      x="${calibration['sensor_kit_base_link']['camera_rear/camera_link']['x']}"
+      y="${calibration['sensor_kit_base_link']['camera_rear/camera_link']['y']}"
+      z="${calibration['sensor_kit_base_link']['camera_rear/camera_link']['z']}"
+      roll="${calibration['sensor_kit_base_link']['camera_rear/camera_link']['roll']}"
+      pitch="${calibration['sensor_kit_base_link']['camera_rear/camera_link']['pitch']}"
+      yaw="${calibration['sensor_kit_base_link']['camera_rear/camera_link']['yaw']}"
       fps="30"
       width="800"
@@ -112,13 +104,13 @@
     />
     <xacro:monocular_camera_macro
-      name="camera2/camera"
+      name="camera_front_left/camera"
       parent="sensor_kit_base_link"
       namespace=""
-      x="${calibration['sensor_kit_base_link']['camera2/camera_link']['x']}"
-      y="${calibration['sensor_kit_base_link']['camera2/camera_link']['y']}"
-      z="${calibration['sensor_kit_base_link']['camera2/camera_link']['z']}"
-      roll="${calibration['sensor_kit_base_link']['camera2/camera_link']['roll']}"
-      pitch="${calibration['sensor_kit_base_link']['camera2/camera_link']['pitch']}"
-      yaw="${calibration['sensor_kit_base_link']['camera2/camera_link']['yaw']}"
+      x="${calibration['sensor_kit_base_link']['camera_front_left/camera_link']['x']}"
+      y="${calibration['sensor_kit_base_link']['camera_front_left/camera_link']['y']}"
+      z="${calibration['sensor_kit_base_link']['camera_front_left/camera_link']['z']}"
+      roll="${calibration['sensor_kit_base_link']['camera_front_left/camera_link']['roll']}"
+      pitch="${calibration['sensor_kit_base_link']['camera_front_left/camera_link']['pitch']}"
+      yaw="${calibration['sensor_kit_base_link']['camera_front_left/camera_link']['yaw']}"
       fps="30"
       width="800"
@@ -127,13 +119,13 @@
     />
     <xacro:monocular_camera_macro
-      name="camera3/camera"
+      name="camera_front_right/camera"
       parent="sensor_kit_base_link"
       namespace=""
-      x="${calibration['sensor_kit_base_link']['camera3/camera_link']['x']}"
-      y="${calibration['sensor_kit_base_link']['camera3/camera_link']['y']}"
-      z="${calibration['sensor_kit_base_link']['camera3/camera_link']['z']}"
-      roll="${calibration['sensor_kit_base_link']['camera3/camera_link']['roll']}"
-      pitch="${calibration['sensor_kit_base_link']['camera3/camera_link']['pitch']}"
-      yaw="${calibration['sensor_kit_base_link']['camera3/camera_link']['yaw']}"
+      x="${calibration['sensor_kit_base_link']['camera_front_right/camera_link']['x']}"
+      y="${calibration['sensor_kit_base_link']['camera_front_right/camera_link']['y']}"
+      z="${calibration['sensor_kit_base_link']['camera_front_right/camera_link']['z']}"
+      roll="${calibration['sensor_kit_base_link']['camera_front_right/camera_link']['roll']}"
+      pitch="${calibration['sensor_kit_base_link']['camera_front_right/camera_link']['pitch']}"
+      yaw="${calibration['sensor_kit_base_link']['camera_front_right/camera_link']['yaw']}"
       fps="30"
       width="800"
@@ -142,13 +134,13 @@
     />
     <xacro:monocular_camera_macro
-      name="camera4/camera"
+      name="camera_rear_left/camera"
       parent="sensor_kit_base_link"
       namespace=""
-      x="${calibration['sensor_kit_base_link']['camera4/camera_link']['x']}"
-      y="${calibration['sensor_kit_base_link']['camera4/camera_link']['y']}"
-      z="${calibration['sensor_kit_base_link']['camera4/camera_link']['z']}"
-      roll="${calibration['sensor_kit_base_link']['camera4/camera_link']['roll']}"
-      pitch="${calibration['sensor_kit_base_link']['camera4/camera_link']['pitch']}"
-      yaw="${calibration['sensor_kit_base_link']['camera4/camera_link']['yaw']}"
+      x="${calibration['sensor_kit_base_link']['camera_rear_left/camera_link']['x']}"
+      y="${calibration['sensor_kit_base_link']['camera_rear_left/camera_link']['y']}"
+      z="${calibration['sensor_kit_base_link']['camera_rear_left/camera_link']['z']}"
+      roll="${calibration['sensor_kit_base_link']['camera_rear_left/camera_link']['roll']}"
+      pitch="${calibration['sensor_kit_base_link']['camera_rear_left/camera_link']['pitch']}"
+      yaw="${calibration['sensor_kit_base_link']['camera_rear_left/camera_link']['yaw']}"
       fps="30"
       width="800"
@@ -157,13 +149,13 @@
     />
     <xacro:monocular_camera_macro
-      name="camera5/camera"
+      name="camera_rear_right/camera"
       parent="sensor_kit_base_link"
       namespace=""
-      x="${calibration['sensor_kit_base_link']['camera5/camera_link']['x']}"
-      y="${calibration['sensor_kit_base_link']['camera5/camera_link']['y']}"
-      z="${calibration['sensor_kit_base_link']['camera5/camera_link']['z']}"
-      roll="${calibration['sensor_kit_base_link']['camera5/camera_link']['roll']}"
-      pitch="${calibration['sensor_kit_base_link']['camera5/camera_link']['pitch']}"
-      yaw="${calibration['sensor_kit_base_link']['camera5/camera_link']['yaw']}"
+      x="${calibration['sensor_kit_base_link']['camera_rear_right/camera_link']['x']}"
+      y="${calibration['sensor_kit_base_link']['camera_rear_right/camera_link']['y']}"
+      z="${calibration['sensor_kit_base_link']['camera_rear_right/camera_link']['z']}"
+      roll="${calibration['sensor_kit_base_link']['camera_rear_right/camera_link']['roll']}"
+      pitch="${calibration['sensor_kit_base_link']['camera_rear_right/camera_link']['pitch']}"
+      yaw="${calibration['sensor_kit_base_link']['camera_rear_right/camera_link']['yaw']}"
       fps="30"
       width="800"
@@ -173,26 +165,26 @@
     <!-- gnss -->
     <xacro:imu_macro
-      name="gnss"
+      name="adma/gnss"
       parent="sensor_kit_base_link"
       namespace=""
-      x="${calibration['sensor_kit_base_link']['gnss_link']['x']}"
-      y="${calibration['sensor_kit_base_link']['gnss_link']['y']}"
-      z="${calibration['sensor_kit_base_link']['gnss_link']['z']}"
-      roll="${calibration['sensor_kit_base_link']['gnss_link']['roll']}"
-      pitch="${calibration['sensor_kit_base_link']['gnss_link']['pitch']}"
-      yaw="${calibration['sensor_kit_base_link']['gnss_link']['yaw']}"
+      x="${calibration['sensor_kit_base_link']['adma/gnss_link']['x']}"
+      y="${calibration['sensor_kit_base_link']['adma/gnss_link']['y']}"
+      z="${calibration['sensor_kit_base_link']['adma/gnss_link']['z']}"
+      roll="${calibration['sensor_kit_base_link']['adma/gnss_link']['roll']}"
+      pitch="${calibration['sensor_kit_base_link']['adma/gnss_link']['pitch']}"
+      yaw="${calibration['sensor_kit_base_link']['adma/gnss_link']['yaw']}"
       fps="100"
     />
     <!-- imu -->
     <xacro:imu_macro
-      name="tamagawa/imu"
-      parent="sensor_kit_base_link"
+      name="adma/imu"
+      parent="adma/gnss_link"
       namespace=""
-      x="${calibration['sensor_kit_base_link']['tamagawa/imu_link']['x']}"
-      y="${calibration['sensor_kit_base_link']['tamagawa/imu_link']['y']}"
-      z="${calibration['sensor_kit_base_link']['tamagawa/imu_link']['z']}"
-      roll="${calibration['sensor_kit_base_link']['tamagawa/imu_link']['roll']}"
-      pitch="${calibration['sensor_kit_base_link']['tamagawa/imu_link']['pitch']}"
-      yaw="${calibration['sensor_kit_base_link']['tamagawa/imu_link']['yaw']}"
+      x="${calibration['adma/gnss_link']['adma/imu_link']['x']}"
+      y="${calibration['adma/gnss_link']['adma/imu_link']['y']}"
+      z="${calibration['adma/gnss_link']['adma/imu_link']['z']}"
+      roll="${calibration['adma/gnss_link']['adma/imu_link']['roll']}"
+      pitch="${calibration['adma/gnss_link']['adma/imu_link']['pitch']}"
+      yaw="${calibration['adma/gnss_link']['adma/imu_link']['yaw']}"
       fps="100"
     />

File: nissan_leaf_sensor_kit_description/urdf/sensors.xacro (robot description, xacro)
@@ -15,14 +15,3 @@
   />
   <!-- embedded sensors -->
-  <xacro:include filename="$(find velodyne_description)/urdf/VLP-16.urdf.xacro"/>
-  <xacro:VLP-16 parent="base_link" name="velodyne_rear" topic="velodyne_rear/velodyne_points" hz="10" samples="220" gpu="false">
-    <origin
-      xyz="${calibration['base_link']['velodyne_rear_base_link']['x']}
-           ${calibration['base_link']['velodyne_rear_base_link']['y']}
-           ${calibration['base_link']['velodyne_rear_base_link']['z']}"
-      rpy="${calibration['base_link']['velodyne_rear_base_link']['roll']}
-           ${calibration['base_link']['velodyne_rear_base_link']['pitch']}
-           ${calibration['base_link']['velodyne_rear_base_link']['yaw']}"
-    />
-  </xacro:VLP-16>
 </robot>

Commit message: Modified Calibrations, Added front_axle_center_link

File: nissan_leaf_sensor_kit_description/urdf/sensor_kit.xacro (robot description, xacro)
@@ -8,4 +8,5 @@
     <xacro:include filename="$(find ouster_description)/urdf/OS1-64.urdf.xacro"/>
     <xacro:include filename="$(find ouster_description)/urdf/OS2-64.urdf.xacro"/>
+    <xacro:include filename="$(find radar_description)/urdf/radar.xacro"/>
     <xacro:arg name="gpu" default="false"/>
     <xacro:arg name="config_dir" default="$(find nissan_leaf_sensor_kit_description)/config"/>
@@ -17,4 +18,13 @@
     </joint>
     <link name="${sensor_kit_base_link}">
+      <origin rpy="0 0 0" xyz="0 0 0"/>
+    </link>
+    <xacro:property name="front_axle_center_link" default="front_axle_center_link"/>
+    <joint name="${front_axle_center_link}_joint" type="fixed">
+      <origin rpy="0 0 0" xyz="2.7 0 0.29"/>
+      <parent link="base_link"/>
+      <child link="${front_axle_center_link}"/>
+    </joint>
+    <link name="${front_axle_center_link}">
       <origin rpy="0 0 0" xyz="0 0 0"/>
     </link>
@@ -174,5 +184,5 @@
       pitch="${calibration['sensor_kit_base_link']['adma/gnss_link']['pitch']}"
       yaw="${calibration['sensor_kit_base_link']['adma/gnss_link']['yaw']}"
-      fps="100"
+      fps="500"
     />
     <!-- imu -->
@@ -187,5 +197,50 @@
       pitch="${calibration['adma/gnss_link']['adma/imu_link']['pitch']}"
       yaw="${calibration['adma/gnss_link']['adma/imu_link']['yaw']}"
-      fps="100"
+      fps="500"
+    />
+    <!-- radar -->
+    <xacro:radar_macro
+      name="radar_front_left/base_link"
+      parent="front_axle_center_link"
+      namespace=""
+      x="${calibration['front_axle_center_link']['radar_front_left/base_link']['x']}"
+      y="${calibration['front_axle_center_link']['radar_front_left/base_link']['y']}"
+      z="${calibration['front_axle_center_link']['radar_front_left/base_link']['z']}"
+      roll="${calibration['front_axle_center_link']['radar_front_left/base_link']['roll']}"
+      pitch="${calibration['front_axle_center_link']['radar_front_left/base_link']['pitch']}"
+      yaw="${calibration['front_axle_center_link']['radar_front_left/base_link']['yaw']}"
+    />
+    <xacro:radar_macro
+      name="radar_front_right/base_link"
+      parent="front_axle_center_link"
+      namespace=""
+      x="${calibration['front_axle_center_link']['radar_front_right/base_link']['x']}"
+      y="${calibration['front_axle_center_link']['radar_front_right/base_link']['y']}"
+      z="${calibration['front_axle_center_link']['radar_front_right/base_link']['z']}"
+      roll="${calibration['front_axle_center_link']['radar_front_right/base_link']['roll']}"
+      pitch="${calibration['front_axle_center_link']['radar_front_right/base_link']['pitch']}"
+      yaw="${calibration['front_axle_center_link']['radar_front_right/base_link']['yaw']}"
+    />
+    <xacro:radar_macro
+      name="radar_rear_left/base_link"
+      parent="front_axle_center_link"
+      namespace=""
+      x="${calibration['front_axle_center_link']['radar_rear_left/base_link']['x']}"
+      y="${calibration['front_axle_center_link']['radar_rear_left/base_link']['y']}"
+      z="${calibration['front_axle_center_link']['radar_rear_left/base_link']['z']}"
+      roll="${calibration['front_axle_center_link']['radar_rear_left/base_link']['roll']}"
+      pitch="${calibration['front_axle_center_link']['radar_rear_left/base_link']['pitch']}"
+      yaw="${calibration['front_axle_center_link']['radar_rear_left/base_link']['yaw']}"
+    />
+    <xacro:radar_macro
+      name="radar_rear_right/base_link"
+      parent="front_axle_center_link"
+      namespace=""
+      x="${calibration['front_axle_center_link']['radar_rear_right/base_link']['x']}"
+      y="${calibration['front_axle_center_link']['radar_rear_right/base_link']['y']}"
+      z="${calibration['front_axle_center_link']['radar_rear_right/base_link']['z']}"
+      roll="${calibration['front_axle_center_link']['radar_rear_right/base_link']['roll']}"
+      pitch="${calibration['front_axle_center_link']['radar_rear_right/base_link']['pitch']}"
+      yaw="${calibration['front_axle_center_link']['radar_rear_right/base_link']['yaw']}"
     />
   </xacro:macro>
